File: STM32F042F6P6.sch (KiCad schematic (older format))
At the start: 26 parts

Commit message: update,
Parts:
- FB1: renamed from FB?; footprint (none) -> Package_TO_SOT_SMD:SOT-23-5
- J10: renamed from J?; footprint (none) -> Connector_USB:USB_Micro-B_Molex_47346-0001
- J11: renamed from J?; footprint (none) -> Connector_PinHeader_2.54mm:PinHeader_1x04_P2.54mm_Vertical
- U8: renamed from U?; footprint (none) -> Connector_PinHeader_2.54mm:PinHeader_1x03_P2.54mm_Vertical
- gave numbers to parts that had none: 22
Connections:
- net VDD_STM32: no longer U7.5 (VDDA)
- net PA2 renamed USART2_TX
- net PA3 renamed USART2_RX
- new net VDDA: U7.5 (VDDA)
Other:
- moved on the sheet: C20, C21, C22, C23, D10, R26
