File: sdcard_image_tester.sch (KiCad schematic (older format))
At the start: 2 parts

Commit message: update,
Parts:
- added H1, H2, H3, H4: MOUNT_M2.5, MountingHole:MountingHole_2.7mm_M2.5_DIN965, symbol taobao-mounting-hole:MOUNT_M2.5
- gave numbers to parts that had none: 2
Changed lines of the file:
@@
 EESchema Schematic File Version 4
 LIBS:sdcard_image_tester-cache
-LIBS:coil_relay-cache
-LIBS:sdcard_switch-cache
-LIBS:sdcard_reader-cache
+LIBS:STM32F042F6P6-tryout-cache
 EELAYER 26 0
 EELAYER END
@@
 $EndSheet
 $Comp
-L Jumper:SolderJumper_3_Bridged12 JP?
+L Jumper:SolderJumper_3_Bridged12 JP1
 U 1 1 5C1D2B8C
 P 3300 2650
-F 0 "JP?" V 3250 2800 50  0000 L CNN
+F 0 "JP1" V 3250 2800 50  0000 L CNN
 F 1 "SolderJumper_3_Bridged12" V 3300 2800 50  0000 L CNN
 F 2 "Jumper:SolderJumper-3_P2.0mm_Open_TrianglePad1.0x1.5mm_NumberLabels" H 3300 2650 50  0001 C CNN
@@
 $EndComp
 $Comp
-L Jumper:SolderJumper_3_Bridged12 JP?
+L Jumper:SolderJumper_3_Bridged12 JP2
 U 1 1 5C1D2CD9
 P 3550 2750
-F 0 "JP?" V 3500 2900 50  0000 L CNN
+F 0 "JP2" V 3500 2900 50  0000 L CNN
 F 1 "SolderJumper_3_Bridged12" V 3550 2900 50  0000 L CNN
 F 2 "Jumper:SolderJumper-3_P2.0mm_Open_TrianglePad1.0x1.5mm_NumberLabels" H 3550 2750 50  0001 C CNN
@@
 S 5150 2500 850  550
 U 5C2C736E
-F0 "stm32_core" 50
-F1 "stm32_core.sch" 50
+F0 "STM32F042F6P6" 50
+F1 "STM32F042F6P6.sch" 50
 $EndSheet
+$Comp
+L taobao-mounting-hole:MOUNT_M2.5 H1
+U 1 1 5C2C7F9F
+P 5800 6700
+F 0 "H1" H 5900 6746 50  0000 L CNN
+F 1 "MOUNT_M2.5" H 5900 6655 50  0000 L CNN
+F 2 "MountingHole:MountingHole_2.7mm_M2.5_DIN965" H 5800 6700 50  0001 C CNN
+F 3 "~" H 5800 6700 50  0001 C CNN
+	1    5800 6700
+	1    0    0    -1
+$EndComp
+$Comp
+L taobao-mounting-hole:MOUNT_M2.5 H2
+U 1 1 5C2C7FF1
+P 5800 6950
+F 0 "H2" H 5900 6996 50  0000 L CNN
+F 1 "MOUNT_M2.5" H 5900 6905 50  0000 L CNN
+F 2 "MountingHole:MountingHole_2.7mm_M2.5_DIN965" H 5800 6950 50  0001 C CNN
+F 3 "~" H 5800 6950 50  0001 C CNN
+	1    5800 6950
+	1    0    0    -1
+$EndComp
+$Comp
+L taobao-mounting-hole:MOUNT_M2.5 H3
+U 1 1 5C2C809F
+P 5800 7200
+F 0 "H3" H 5900 7246 50  0000 L CNN
+F 1 "MOUNT_M2.5" H 5900 7155 50  0000 L CNN
+F 2 "MountingHole:MountingHole_2.7mm_M2.5_DIN965" H 5800 7200 50  0001 C CNN
+F 3 "~" H 5800 7200 50  0001 C CNN
+	1    5800 7200
+	1    0    0    -1
+$EndComp
+$Comp
+L taobao-mounting-hole:MOUNT_M2.5 H4
+U 1 1 5C2C80A5
+P 5800 7450
+F 0 "H4" H 5900 7496 50  0000 L CNN
+F 1 "MOUNT_M2.5" H 5900 7405 50  0000 L CNN
+F 2 "MountingHole:MountingHole_2.7mm_M2.5_DIN965" H 5800 7450 50  0001 C CNN
+F 3 "~" H 5800 7450 50  0001 C CNN
+	1    5800 7450
+	1    0    0    -1
+$EndComp
 $EndSCHEMATC

Commit message: update,
Parts:
- removed JP1, JP2: SolderJumper_3_Bridged12, Jumper:SolderJumper-3_P2.0mm_Open_TrianglePad1.0x1.5mm_NumberLabels, symbol Jumper:SolderJumper_3_Bridged12
Changed lines of the file:
@@
 EESchema Schematic File Version 4
 LIBS:sdcard_image_tester-cache
-LIBS:STM32F042F6P6-tryout-cache
 EELAYER 26 0
 EELAYER END
@@
 $EndDescr
 $Sheet
-S 6250 2500 850  550
+S 5000 2550 850  550
 U 5C16890A
 F0 "coil_relay" 50
 F1 "coil_relay.sch" 50
-F2 "R1_CONTROL" I L 6250 2650 50
-F3 "R2_CONTROL" I L 6250 2750 50
+F2 "R1_CONTROL" I L 5000 2700 50
+F3 "R2_CONTROL" I L 5000 2800 50
 $EndSheet
 $Sheet
-S 8250 3450 800  1550
+S 7000 3400 800  1550
 U 5C17CDA9
 F0 "sdcard_reader" 50
 F1 "sdcard_reader.sch" 50
-F2 "READER_DAT2" I L 8250 3550 50
-F3 "READER_DAT3" I L 8250 3650 50
-F4 "READER_CMD" I L 8250 3750 50
-F5 "READER_VDD" I L 8250 3850 50
-F6 "READER_CLK" I L 8250 3950 50
-F7 "READER_VSS" I L 8250 4050 50
-F8 "READER_DAT0" I L 8250 4150 50
-F9 "READER_DAT1" I L 8250 4250 50
-F10 "READER_DET" I L 8250 4350 50
+F2 "READER_DAT2" I L 7000 3500 50
+F3 "READER_DAT3" I L 7000 3600 50
+F4 "READER_CMD" I L 7000 3700 50
+F5 "READER_VDD" I L 7000 3800 50
+F6 "READER_CLK" I L 7000 3900 50
+F7 "READER_VSS" I L 7000 4000 50
+F8 "READER_DAT0" I L 7000 4100 50
+F9 "READER_DAT1" I L 7000 4200 50
+F10 "READER_DET" I L 7000 4300 50
 $EndSheet
 Wire Wire Line
-	7800 3550 8250 3550
+	6550 3500 7000 3500
 Wire Wire Line
-	7800 3650 8250 3650
+	6550 3600 7000 3600
 Wire Wire Line
-	7800 3750 8250 3750
+	6550 3700 7000 3700
 Wire Wire Line
-	7800 3850 8250 3850
+	6550 3800 7000 3800
 Wire Wire Line
-	7800 3950 8250 3950
+	6550 3900 7000 3900
 Wire Wire Line
-	7800 4050 8250 4050
+	6550 4000 7000 4000
 Wire Wire Line
-	7800 4150 8250 4150
+	6550 4100 7000 4100
 Wire Wire Line
-	7800 4250 8250 4250
+	6550 4200 7000 4200
 $Sheet
 S 2050 2500 850  550
@@
 F3 "CH340_TXD" O R 2900 2750 50
 $EndSheet
-$Comp
-L Jumper:SolderJumper_3_Bridged12 JP1
-U 1 1 5C1D2B8C
-P 3300 2650
-F 0 "JP1" V 3250 2800 50  0000 L CNN
-F 1 "SolderJumper_3_Bridged12" V 3300 2800 50  0000 L CNN
-F 2 "Jumper:SolderJumper-3_P2.0mm_Open_TrianglePad1.0x1.5mm_NumberLabels" H 3300 2650 50  0001 C CNN
-F 3 "~" H 3300 2650 50  0001 C CNN
-	1    3300 2650
-	0    1    1    0
-$EndComp
-$Comp
-L Jumper:SolderJumper_3_Bridged12 JP2
-U 1 1 5C1D2CD9
-P 3550 2750
-F 0 "JP2" V 3500 2900 50  0000 L CNN
-F 1 "SolderJumper_3_Bridged12" V 3550 2900 50  0000 L CNN
-F 2 "Jumper:SolderJumper-3_P2.0mm_Open_TrianglePad1.0x1.5mm_NumberLabels" H 3550 2750 50  0001 C CNN
-F 3 "~" H 3550 2750 50  0001 C CNN
-	1    3550 2750
-	0    1    1    0
-$EndComp
-Wire Wire Line
-	2900 2650 3150 2650
-Wire Wire Line
-	2900 2750 3400 2750
-Wire Wire Line
-	3800 2500 3550 2500
-Wire Wire Line
-	3550 2500 3550 2550
-Wire Wire Line
-	3850 2400 3300 2400
-Wire Wire Line
-	3300 2400 3300 2450
-Wire Wire Line
-	3300 2850 3300 3050
-Wire Wire Line
-	3300 3050 3800 3050
-Wire Wire Line
-	3550 2950 3550 3150
-Wire Wire Line
-	3550 3150 3850 3150
 $Sheet
-S 6250 3400 1550 2300
+S 5000 3350 1550 2300
 U 5C168465
 F0 "sdcard_switch" 50
 F1 "sdcard_switch.sch" 50
-F2 "PC_DAT2" I R 7800 3550 50
-F3 "PC_DAT3" I R 7800 3650 50
-F4 "PC_CMD" I R 7800 3750 50
-F5 "PC_VDD" I R 7800 3850 50
-F6 "PC_CLK" I R 7800 3950 50
-F7 "PC_VSS" I R 7800 4050 50
-F8 "PC_DAT0" I R 7800 4150 50
-F9 "PC_DAT1" I R 7800 4250 50
-F10 "DUT_DAT2" I R 7800 4500 50
-F11 "DUT_DAT3" I R 7800 4600 50
-F12 "DUT_CMD" I R 7800 4700 50
-F13 "DUT_VDD" I R 7800 4800 50
-F14 "DUT_CLK" I R 7800 4900 50
-F15 "DUT_VSS" I R 7800 5000 50
-F16 "DUT_DAT0" I R 7800 5100 50
-F17 "DUT_DAT1" I R 7800 5200 50
-F18 "HOSTSELECT" I L 6250 3550 50
-$EndSheet
-Wire Wire Line
-	3800 2500 3800 3050
-Wire Wire Line
-	3850 2400 3850 3150
-$Sheet
-S 5150 2500 850  550
-U 5C2C736E
-F0 "STM32F042F6P6" 50
-F1 "STM32F042F6P6.sch" 50
+F2 "PC_DAT2" I R 6550 3500 50
+F3 "PC_DAT3" I R 6550 3600 50
+F4 "PC_CMD" I R 6550 3700 50
+F5 "PC_VDD" I R 6550 3800 50
+F6 "PC_CLK" I R 6550 3900 50
+F7 "PC_VSS" I R 6550 4000 50
+F8 "PC_DAT0" I R 6550 4100 50
+F9 "PC_DAT1" I R 6550 4200 50
+F10 "DUT_DAT2" I R 6550 4450 50
+F11 "DUT_DAT3" I R 6550 4550 50
+F12 "DUT_CMD" I R 6550 4650 50
+F13 "DUT_VDD" I R 6550 4750 50
+F14 "DUT_CLK" I R 6550 4850 50
+F15 "DUT_VSS" I R 6550 4950 50
+F16 "DUT_DAT0" I R 6550 5050 50
+F17 "DUT_DAT1" I R 6550 5150 50
+F18 "HOSTSELECT" I L 5000 3500 50
 $EndSheet
 $Comp
@@
 	1    0    0    -1
 $EndComp
+$Sheet
+S 3050 2500 1250 850
+U 5C2C736E
+F0 "STM32F042F6P6" 50
+F1 "STM32F042F6P6.sch" 50
+F2 "USART2_TX" O L 3050 2650 50
+F3 "USART2_RX" I L 3050 2750 50
+F4 "PA6" O R 4300 2800 50
+F5 "PA7" O R 4300 2700 50
+F6 "PA5" O R 4300 2900 50
+$EndSheet
+Wire Wire Line
+	2900 2650 3050 2650
+Wire Wire Line
+	2900 2750 3050 2750
+Wire Wire Line
+	4300 2700 5000 2700
+Wire Wire Line
+	4300 2800 5000 2800
+Wire Wire Line
+	4300 2900 4600 2900
+Wire Wire Line
+	4600 2900 4600 3500
+Wire Wire Line
+	4600 3500 5000 3500
 $EndSCHEMATC
