File: sdcard_image_tester.kicad_pcb (KiCad board)
At the start: 2 copper layers, 43 x 75 mm, 1 part

Commit message: update,
Parts:
- added C1: CP4.7uf,50V, Capacitor_SMD:CP_Elec_4x5.3, F.Cu at (15.9, 152.6)
- added C10: C22pf,0603, Capacitor_SMD:C_0603_1608Metric_Pad1.05x0.95mm_HandSolder, F.Cu at (94.1, 140.4)
- added C11: C102,0603, Capacitor_SMD:C_0603_1608Metric_Pad1.05x0.95mm_HandSolder, F.Cu at (94.1, 138.9)
- added C12: CP22uf,16V, Capacitor_SMD:CP_Elec_4x5.3, F.Cu at (56.6, 146.6)
- added C13: C106,0603, Capacitor_SMD:C_0603_1608Metric_Pad1.05x0.95mm_HandSolder, F.Cu at (68.4, 149.3)
- added C14: C103,0603, Capacitor_SMD:C_0603_1608Metric_Pad1.05x0.95mm_HandSolder, F.Cu at (75.7, 144.3)
- added C15: C104,0603, Capacitor_SMD:C_0603_1608Metric_Pad1.05x0.95mm_HandSolder, F.Cu at (71.1, 141.3)
- added C16: C475,0603, Capacitor_SMD:C_0603_1608Metric_Pad1.05x0.95mm_HandSolder, F.Cu at (74.4, 142.8)
- added C17: C22pf,0603, Capacitor_SMD:C_0603_1608Metric_Pad1.05x0.95mm_HandSolder, F.Cu at (72.3, 145.8)
- added C18: C22pf,0603, Capacitor_SMD:C_0603_1608Metric_Pad1.05x0.95mm_HandSolder, F.Cu at (69.0, 147.8)
- added C19: C104,0603, Capacitor_SMD:C_0603_1608Metric_Pad1.05x0.95mm_HandSolder, F.Cu at (72.3, 144.3)
- added C2: C22pf,0603, Capacitor_SMD:C_0603_1608Metric_Pad1.05x0.95mm_HandSolder, F.Cu at (84.6, 114.9)
- added C20: C103,0603, Capacitor_SMD:C_0603_1608Metric_Pad1.05x0.95mm_HandSolder, F.Cu at (69.0, 146.3)
- added C21: C105,0603, Capacitor_SMD:C_0603_1608Metric_Pad1.05x0.95mm_HandSolder, F.Cu at (75.9, 139.2)
- added C22: C475,0603, Capacitor_SMD:C_0603_1608Metric_Pad1.05x0.95mm_HandSolder, F.Cu at (74.4, 141.3)
- added C23: C104,0603, Capacitor_SMD:C_0603_1608Metric_Pad1.05x0.95mm_HandSolder, F.Cu at (71.1, 142.8)
- added C3: C22pf,0603, Capacitor_SMD:C_0603_1608Metric_Pad1.05x0.95mm_HandSolder, F.Cu at (68.5, 125.7)
- added C4: C104,0603, Capacitor_SMD:C_0603_1608Metric_Pad1.05x0.95mm_HandSolder, F.Cu at (73.7, 124.1)
- added C5: C104,0603, Capacitor_SMD:C_0603_1608Metric_Pad1.05x0.95mm_HandSolder, F.Cu at (84.6, 116.4)
- added C6: C104,0603, Capacitor_SMD:C_0603_1608Metric_Pad1.05x0.95mm_HandSolder, F.Cu at (73.7, 122.6)
- added C7: C226,6.3v,0603, Capacitor_SMD:C_0603_1608Metric_Pad1.05x0.95mm_HandSolder, F.Cu at (90.7, 143.0)
- added C8: C104,0603, Capacitor_SMD:C_0603_1608Metric_Pad1.05x0.95mm_HandSolder, F.Cu at (95.0, 137.0)
- added C9: C22pf,0603, Capacitor_SMD:C_0603_1608Metric_Pad1.05x0.95mm_HandSolder, F.Cu at (90.7, 141.5)
- added D1: RELAY_STATUS, LED_SMD:LED_0805_2012Metric_Castellated, F.Cu at (26.2, 154.7)
- added D10: LED_GREEN,0603, LED_SMD:LED_0603_1608Metric_Pad1.05x0.95mm_HandSolder, F.Cu at (61.7, 149.3)
- added D2: 1N4148, Diode_SMD:D_SOD-323_HandSoldering, F.Cu at (47.6, 137.9)
- added D3: 3V3_STATUS, LED_SMD:LED_0805_2012Metric_Castellated, F.Cu at (22.3, 154.7)
- added D4: RELAY_STATUS, LED_SMD:LED_0805_2012Metric_Castellated, F.Cu at (18.5, 156.0)
- added D5: 1N4148, Diode_SMD:D_SOD-323_HandSoldering, F.Cu at (14.5, 156.0)
- added D6: LED_GREEN,0603, LED_SMD:LED_0603_1608Metric_Pad1.05x0.95mm_HandSolder, F.Cu at (84.6, 110.8)
- added D7: LED_ORANGE,0603, LED_SMD:LED_0603_1608Metric_Pad1.05x0.95mm_HandSolder, F.Cu at (30.1, 129.1)
- added D8: LED_GREEN,0603, LED_SMD:LED_0603_1608Metric_Pad1.05x0.95mm_HandSolder, F.Cu at (49.3, 110.8)
- added D9: LED_GREEN,0603, LED_SMD:LED_0603_1608Metric_Pad1.05x0.95mm_HandSolder, F.Cu at (54.9, 149.8)
- added FB1: UPZ1608E221-2R2TF, Package_TO_SOT_SMD:SOT-23-5, F.Cu at (-14.4, 121.0)
- added H1: MOUNT_M2.5, MountingHole:MountingHole_2.7mm_M2.5_DIN965, F.Cu at (99.3, 117.9)
- added H2: MOUNT_M2.5, MountingHole:MountingHole_2.7mm_M2.5_DIN965, F.Cu at (99.3, 112.6)
- added H3: MOUNT_M2.5, MountingHole:MountingHole_2.7mm_M2.5_DIN965, F.Cu at (94.0, 112.6)
- added H4: MOUNT_M2.5, MountingHole:MountingHole_2.7mm_M2.5_DIN965, F.Cu at (94.0, 117.9)
- added J1: Conn_01x02, Connector_PinHeader_1.27mm:PinHeader_1x02_P1.27mm_Vertical, F.Cu at (31.7, 151.4)
- added J10: USB_B_Micro, Connector_USB:USB_Micro-B_Molex_47346-0001, F.Cu at (-11.7, 115.2)
- added J11: Conn_02x02_Odd_Even, Connector_PinHeader_2.54mm:PinHeader_1x04_P2.54mm_Vertical, F.Cu at (-18.2, 114.3)
- added J2: Conn_02x03_Odd_Even, Connector_PinHeader_2.54mm:PinHeader_2x03_P2.54mm_Vertical_SMD, F.Cu at (39.6, 141.3)
- added J3: Conn_02x03_Odd_Even, Connector_PinHeader_2.54mm:PinHeader_2x03_P2.54mm_Vertical_SMD, F.Cu at (39.6, 150.0)
- added J4: USB_B_Micro, Connector_USB:USB_Micro-B_Molex-105017-0001, F.Cu at (62.4, 122.8)
- added J5: Conn_01x09, Connector_FFC-FPC:TE_84953-9_1x09-1MP_P1.0mm_Horizontal, F.Cu at (66.9, 113.3)
- added J6: USB_B_Mini, Connector_USB:USB_Micro-B_Molex-105017-0001, F.Cu at (97.8, 132.6)
- added J7: Conn_01x09, Connector_PinHeader_1.27mm:PinHeader_1x09_P1.27mm_Vertical, F.Cu at (82.2, 131.3)
- added J8: TO_PC, Connector_FFC-FPC:TE_84952-8_1x08-1MP_P1.0mm_Horizontal, F.Cu at (39.1, 113.3)
- added J9: TO_DUT, Connector_FFC-FPC:Hirose_FH12-8S-0.5SH_1x08-1MP_P0.50mm_Horizontal, F.Cu at (35.7, 123.4)
- added JP3: SolderJumper_2_Open, Jumper:SolderJumper-2_P1.3mm_Open_TrianglePad1.0x1.5mm, F.Cu at (84.6, 112.9)
- added JP4: SolderJumper_2_Open, Jumper:SolderJumper-2_P1.3mm_Open_TrianglePad1.0x1.5mm, F.Cu at (90.7, 139.5)
- added K1: A5W-K, Package_DIP:DIP-10_W7.62mm_LongPads, F.Cu at (14.0, 138.5)
- added K2: A5W-K, Package_DIP:DIP-10_W7.62mm_LongPads, F.Cu at (24.6, 138.5)
- added Q1: 2N3904(1AM), Package_TO_SOT_SMD:SOT-23_Handsoldering, F.Cu at (22.0, 152.0)
- added Q2: 2N3904(1AM), Package_TO_SOT_SMD:SOT-23_Handsoldering, F.Cu at (27.4, 152.0)
- added R1: 102, Resistor_SMD:R_0805_2012Metric_Pad1.15x1.40mm_HandSolder, F.Cu at (26.0, 156.7)
- added R10: R102,0603, Resistor_SMD:R_0603_1608Metric_Pad1.05x0.95mm_HandSolder, F.Cu at (73.7, 121.1)
- added R11: R103,0603, Resistor_SMD:R_0603_1608Metric_Pad1.05x0.95mm_HandSolder, F.Cu at (77.1, 122.7)
- added R12: R103,0603, Resistor_SMD:R_0603_1608Metric_Pad1.05x0.95mm_HandSolder, F.Cu at (77.1, 121.2)
- added R13: R473,0603, Resistor_SMD:R_0603_1608Metric_Pad1.05x0.95mm_HandSolder, F.Cu at (78.5, 125.7)
- added R14: R473,0603, Resistor_SMD:R_0603_1608Metric_Pad1.05x0.95mm_HandSolder, F.Cu at (78.5, 124.2)
- added R15: R473,0603, Resistor_SMD:R_0603_1608Metric_Pad1.05x0.95mm_HandSolder, F.Cu at (84.6, 119.4)
- added R16: R473,0603, Resistor_SMD:R_0603_1608Metric_Pad1.05x0.95mm_HandSolder, F.Cu at (80.4, 122.7)
- added R17: R473,0603, Resistor_SMD:R_0603_1608Metric_Pad1.05x0.95mm_HandSolder, F.Cu at (71.8, 125.7)
- added R18: R473,0603, Resistor_SMD:R_0603_1608Metric_Pad1.05x0.95mm_HandSolder, F.Cu at (80.4, 121.2)
- added R19: R103,0603, Resistor_SMD:R_0603_1608Metric_Pad1.05x0.95mm_HandSolder, F.Cu at (17.5, 133.1)
- added R2: 102, Resistor_SMD:R_0805_2012Metric_Pad1.15x1.40mm_HandSolder, F.Cu at (22.3, 156.7)
- added R20: R103,0603, Resistor_SMD:R_0603_1608Metric_Pad1.05x0.95mm_HandSolder, F.Cu at (14.2, 133.1)
- added R21: R102,0603, Resistor_SMD:R_0603_1608Metric_Pad1.05x0.95mm_HandSolder, F.Cu at (20.9, 133.1)
- added R22: R102,0603, Resistor_SMD:R_0603_1608Metric_Pad1.05x0.95mm_HandSolder, F.Cu at (24.2, 133.1)
- added R23: R103,0603, Resistor_SMD:R_0603_1608Metric_Pad1.05x0.95mm_HandSolder, F.Cu at (69.0, 144.8)
- added R24: R104,0603, Resistor_SMD:R_0603_1608Metric_Pad1.05x0.95mm_HandSolder, F.Cu at (65.0, 149.3)
- added R25: R104,0603, Resistor_SMD:R_0603_1608Metric_Pad1.05x0.95mm_HandSolder, F.Cu at (58.3, 149.8)
- added R26: R102,0603, Resistor_SMD:R_0603_1608Metric_Pad1.05x0.95mm_HandSolder, F.Cu at (75.9, 137.7)
- added R3: 103, Resistor_SMD:R_0805_2012Metric_Pad1.15x1.40mm_HandSolder, F.Cu at (47.4, 143.7)
- added R4: 511, Resistor_SMD:R_0805_2012Metric_Pad1.15x1.40mm_HandSolder, F.Cu at (30.0, 155.4)
- added R5: 102, Resistor_SMD:R_0805_2012Metric_Pad1.15x1.40mm_HandSolder, F.Cu at (33.7, 155.4)
- added R6: 102, Resistor_SMD:R_0805_2012Metric_Pad1.15x1.40mm_HandSolder, F.Cu at (47.4, 139.8)
- added R7: 103, Resistor_SMD:R_0805_2012Metric_Pad1.15x1.40mm_HandSolder, F.Cu at (47.4, 141.8)
- added R8: R220,0603, Resistor_SMD:R_0603_1608Metric_Pad1.05x0.95mm_HandSolder, F.Cu at (84.6, 117.9)
- added R9: R220,0603, Resistor_SMD:R_0603_1608Metric_Pad1.05x0.95mm_HandSolder, F.Cu at (75.2, 125.6)
- added SDC1: TF_CARD_SOCKET,SELF_EJECT, footprint-lib:SUNTECH_ST-TF-003A, F.Cu at (20.3, 116.6)
- added TP1: VSD, TestPoint:TestPoint_Pad_D1.0mm, F.Cu at (29.4, 130.9)
- added TP2: HS, TestPoint:TestPoint_Pad_D1.0mm, F.Cu at (32.8, 129.3)
- added TP3: G, TestPoint:TestPoint_Pad_D1.0mm, F.Cu at (41.8, 121.4)
- added U1: GL827L, Package_SO:SSOP-28_3.9x9.9mm_P0.635mm, F.Cu at (79.4, 115.2)
- added U2: CH340T(SSOP20W), Package_SO:SSOP-20_5.3x7.2mm_P0.65mm, F.Cu at (88.6, 134.2)
- added U3: SN74CBT3257D, Package_SO:TSSOP-16_4.4x5mm_P0.65mm, F.Cu at (16.5, 129.5)
- added U4: SN74CBT3257D, Package_SO:TSSOP-16_4.4x5mm_P0.65mm, F.Cu at (24.4, 129.5)
- added U5: AMS1117-3.3, Package_TO_SOT_SMD:SOT-223-3_TabPin2, F.Cu at (57.6, 140.5)
- added U6: USBLC6-2SC6, Package_TO_SOT_SMD:SOT-23-6_Handsoldering, F.Cu at (71.8, 138.7)
- added U7: STM32F042F6P6, Package_SO:SSOP-20_4.4x6.5mm_P0.65mm, F.Cu at (65.7, 140.5)
- added U8: swd-pinsocket, Connector_PinHeader_2.54mm:PinHeader_1x03_P2.54mm_Vertical, F.Cu at (-5.27, 114.3)
- added Y1: O_12M,3225, Oscillator:Oscillator_SMD_Abracon_ASE-4Pin_3.2x2.5mm_HandSoldering, F.Cu at (69.4, 122.7)
- added Y2: O_12M,3225, Oscillator:Oscillator_SMD_Abracon_ASE-4Pin_3.2x2.5mm_HandSoldering, F.Cu at (86.4, 140.4)
- added Y3: O_8M,3225, Oscillator:Oscillator_SMD_Abracon_ASE-4Pin_3.2x2.5mm_HandSoldering, F.Cu at (64.7, 146.3)

Commit message: update,
Parts:
- removed mouse-bite-2mm-slot: VAL**, Panelization.pretty:mouse-bite-2mm-slot
Other:
- board size 43 x 75 mm -> 41 x 75 mm
Changed lines of the file:
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@@
     (tracks 0)
     (zones 0)
-    (modules 97)
+    (modules 96)
     (nets 116)
   )
@@
     (38 B.Mask user)
     (39 F.Mask user)
-    (40 Dwgs.User user)
+    (40 Dwgs.User user hide)
     (41 Cmts.User user)
     (42 Eco1.User user)
@@
     (pad Hole np_thru_hole circle (at 4.32 5.17) (size 0.9 0.9) (drill 0.9) (layers *.Cu *.Mask F.SilkS))
   )
-  (module Panelization.pretty:mouse-bite-2mm-slot (layer F.Cu)
-    (at 36 14 90)
-    (fp_text reference mouse-bite-2mm-slot (at 0 -2 90) (layer F.SilkS) hide
-      (effects (font (size 1 1) (thickness 0.2)))
-    )
-    (fp_text value VAL** (at 0 2.1 90) (layer F.SilkS) hide
-      (effects (font (size 1 1) (thickness 0.2)))
-    )
-    (fp_line (start 2 0) (end 2 0) (layer Eco1.User) (width 2))
-    (fp_line (start -2 0) (end -2 0) (layer Eco1.User) (width 2))
-    (fp_circle (center -2 0) (end -2 -0.06) (layer Dwgs.User) (width 0.05))
-    (fp_circle (center 2 0) (end 2.06 0) (layer Dwgs.User) (width 0.05))
-    (fp_arc (start 2 0) (end 2 1) (angle 180) (layer F.SilkS) (width 0.1))
-    (fp_arc (start -2 0) (end -2 -1) (angle 180) (layer F.SilkS) (width 0.1))
-    (pad "" np_thru_hole circle (at 0.75 0.75 90) (size 0.5 0.5) (drill 0.5) (layers *.Cu *.Mask))
-    (pad "" np_thru_hole circle (at -0.75 0.75 90) (size 0.5 0.5) (drill 0.5) (layers *.Cu *.Mask))
-    (pad "" np_thru_hole circle (at -0.75 -0.75 90) (size 0.5 0.5) (drill 0.5) (layers *.Cu *.Mask))
-    (pad "" np_thru_hole circle (at 0.75 -0.75 90) (size 0.5 0.5) (drill 0.5) (layers *.Cu *.Mask))
-    (pad "" np_thru_hole circle (at 0 0.75 90) (size 0.5 0.5) (drill 0.5) (layers *.Cu *.Mask))
-    (pad "" np_thru_hole circle (at 0 -0.75 90) (size 0.5 0.5) (drill 0.5) (layers *.Cu *.Mask))
-  )
+  (gr_line (start 35 12) (end 35 10) (layer Edge.Cuts) (width 0.15))
+  (gr_arc (start 34 12) (end 33 12) (angle -180) (layer Edge.Cuts) (width 0.15))
+  (gr_arc (start 34 16) (end 35 16) (angle -180) (layer Edge.Cuts) (width 0.15))
+  (gr_line (start 41 10) (end 35 10) (layer Edge.Cuts) (width 0.15))
+  (gr_line (start 41 17) (end 41 10) (layer Edge.Cuts) (width 0.15))
+  (gr_line (start 35 17) (end 41 17) (layer Edge.Cuts) (width 0.15))
+  (gr_line (start 35 16) (end 35 17) (layer Edge.Cuts) (width 0.15))
   (gr_line (start 0 100) (end 0 0) (layer Dwgs.User) (width 0.2))
   (gr_line (start 100 100) (end 0 100) (layer Dwgs.User) (width 0.2))
   (gr_line (start 100 0) (end 100 100) (layer Dwgs.User) (width 0.2))
   (gr_line (start 0 0) (end 100 0) (layer Dwgs.User) (width 0.2))
-  (gr_line (start 35 2.5) (end 35 12) (layer Edge.Cuts) (width 0.15))
-  (gr_arc (start 32.5 2.5) (end 35 2.5) (angle -90) (layer Edge.Cuts) (width 0.15))
-  (gr_line (start 37 12) (end 37 10) (layer Edge.Cuts) (width 0.15))
-  (gr_arc (start 36 12) (end 35 12) (angle -180) (layer Edge.Cuts) (width 0.15))
-  (gr_arc (start 36 16) (end 37 16) (angle -180) (layer Edge.Cuts) (width 0.15))
-  (gr_line (start 43 10) (end 37 10) (layer Edge.Cuts) (width 0.15))
-  (gr_line (start 43 17) (end 43 10) (layer Edge.Cuts) (width 0.15))
-  (gr_line (start 37 17) (end 43 17) (layer Edge.Cuts) (width 0.15))
-  (gr_line (start 37 16) (end 37 17) (layer Edge.Cuts) (width 0.15))
+  (gr_line (start 33 2.5) (end 33 12) (layer Edge.Cuts) (width 0.15))
+  (gr_arc (start 30.5 2.5) (end 33 2.5) (angle -90) (layer Edge.Cuts) (width 0.15))
   (dimension 35 (width 0.3) (layer Dwgs.User)
     (gr_text "35.000 mm" (at 17.5 -12.1) (layer Dwgs.User)
@@
   (gr_arc (start 2.5 2.5) (end 2.5 0) (angle -90) (layer Edge.Cuts) (width 0.15))
   (gr_arc (start 2.5 72.5) (end 0 72.5) (angle -90) (layer Edge.Cuts) (width 0.15))
-  (gr_arc (start 32.5 72.5) (end 32.5 75) (angle -90) (layer Edge.Cuts) (width 0.15))
-  (gr_line (start 32.5 0) (end 2.5 0) (layer Edge.Cuts) (width 0.15))
-  (gr_line (start 35 72.5) (end 35 16) (layer Edge.Cuts) (width 0.15))
-  (gr_line (start 2.5 75) (end 32.5 75) (layer Edge.Cuts) (width 0.15))
+  (gr_arc (start 30.5 72.5) (end 30.5 75) (angle -90) (layer Edge.Cuts) (width 0.15))
+  (gr_line (start 30.5 0) (end 2.5 0) (layer Edge.Cuts) (width 0.15))
+  (gr_line (start 33 72.5) (end 33 16) (layer Edge.Cuts) (width 0.15))
+  (gr_line (start 2.5 75) (end 30.5 75) (layer Edge.Cuts) (width 0.15))
   (gr_line (start 0 2.5) (end 0 72.5) (layer Edge.Cuts) (width 0.15))
 )
